Commit message: Adding the RP Lidar sensor to Gazebo model

File: simulation_ws/src/deepracer_simulation/urdf/racecar.xacro (robot description, xacro)
@@ -201,4 +201,30 @@
     <axis xyz="0 0 1" />
   </joint>
+<joint name="rplidar_joint" type="fixed">
+    <axis xyz="0 1 0" />
+    <origin xyz="0.02 0 0.058" rpy="0 0 3.14"/>
+    <parent link="base_link"/>
+    <child link="laser"/>
+  </joint>
+  <!-- rplidar Laser -->
+  <link name="laser">
+    <collision>
+      <origin xyz="0 0 0" rpy="1.5707 0 4.71"/>
+      <geometry>
+        <mesh filename="package://deepracer_simulation/meshes/rplidar.dae" scale="0.001 0.001 0.001" />
+      </geometry>
+    </collision>
+    <visual>
+      <origin xyz="0 0 0" rpy="1.5707 0 4.71"/>
+      <geometry>
+        <mesh filename="package://deepracer_simulation/meshes/rplidar.dae" scale="0.001 0.001 0.001" />
+      </geometry>
+    </visual>
+    <inertial>
+      <mass value="1e-5" />
+      <origin xyz="0 0 0" rpy="1.5707 0 4.71"/>
+      <inertia ixx="0" ixy="0" ixz="0" iyy="0" iyz="0" izz="0" />
+    </inertial>
+  </link>
   <!-- Add the remaining xacros -->
   <xacro:include filename="$(find deepracer_simulation)/urdf/racecar.gazebo" />
